Commit message: Update map, robot speed and keyboard control

File: urdf/robot_core.xacro (robot description, xacro)
@@ -74,5 +74,5 @@
         <child link="left_wheel"/>
         <origin xyz="0 ${wheel_offset_y} 0" rpy="1.570795 0 0" />
-        <axis xyz="0 0 1"/>
+        <axis xyz="0 0 -1"/>
     </joint>
     <link name="left_wheel">
